Commit message: finished robot drive train urdf

File: src/crobot_description/description/depth_camera.xacro (robot description, xacro)
@@ -4,5 +4,5 @@
         <parent link="chassis"/>
         <child link="camera_link"/>
-        <origin xyz="0.305 0 0.08" rpy="0 0 0"/>
+        <origin xyz="0.305 0 0.038" rpy="0 ${pi/10} 0"/>
     </joint>
     <link name="camera_link">

File: src/crobot_description/description/robot.urdf.xacro (robot description, xacro)
@@ -3,6 +3,6 @@
     <xacro:arg name="use_ros2_control" default="true"/>
     <xacro:arg name="sim_mode" default="false"/>
-    <!-- <xacro:include filename="robot_core.xacro"/> -->
-    <xacro:include filename="drivetrain/robot.urdf"/>
+    <xacro:include filename="robot_core.xacro"/>
+    <!-- <xacro:include filename="drivetrain/robot.urdf"/> -->
     <xacro:if value="$(arg use_ros2_control)">
         <xacro:include filename="ros2_control.xacro"/>

File: src/crobot_description/description/robot_core.xacro (robot description, xacro)
@@ -19,22 +19,78 @@
         <parent link="base_link"/>
         <child link="chassis"/>
-        <origin xyz="-0.15 0 0"/>
+        <origin xyz="-0.144 0 0"/>
     </joint>
     <link name="chassis">
         <visual>
-            <origin xyz="0.15 0 0.075"/>
-            <geometry>
-                <box size="0.3 0.3 0.15"/>
-            </geometry>
-            <material name="white"/>
-        </visual>
-        <collision>
-            <origin xyz="0.15 0 0.075"/>
-            <geometry>
-                <box size="0.3 0.3 0.15"/>
-            </geometry>
-        </collision>
-        <xacro:inertial_box mass="0.5" x="0.3" y="0.3" z="0.15">
-            <origin xyz="0.15 0 0.075" rpy="0 0 0"/>
+            <origin xyz="0.144 0 0.038"/>
+            <geometry>
+                <box size="0.096 0.168 0.048"/>
+            </geometry>
+            <material name="white"/>
+        </visual>
+        <visual>
+            <origin xyz="0.144 0.09 0.038"/>
+            <geometry>
+                <box size="0.288 0.012 0.048"/>
+            </geometry>
+            <material name="white"/>
+        </visual>
+        <visual>
+            <origin xyz="0.144 -0.09 0.038"/>
+            <geometry>
+                <box size="0.288 0.012 0.048"/>
+            </geometry>
+            <material name="white"/>
+        </visual>
+        <visual>
+            <origin xyz="0.00125 0.11995 0.038"/>
+            <geometry>
+                <box size="0.0025 0.0479 0.048"/>
+            </geometry>
+            <material name="white"/>
+        </visual>
+        <visual>
+            <origin xyz="0.00125 -0.11995 0.038"/>
+            <geometry>
+                <box size="0.0025 0.0479 0.048"/>
+            </geometry>
+            <material name="white"/>
+        </visual>
+        <visual>
+            <origin xyz="0.28675 0.11995 0.038"/>
+            <geometry>
+                <box size="0.0025 0.0479 0.048"/>
+            </geometry>
+            <material name="white"/>
+        </visual>
+        <visual>
+            <origin xyz="0.28675 -0.11995 0.038"/>
+            <geometry>
+                <box size="0.0025 0.0479 0.048"/>
+            </geometry>
+            <material name="white"/>
+        </visual>
+        <visual>
+            <origin xyz="0.144 0.14515 0.038"/>
+            <geometry>
+                <box size="0.288 0.0025 0.048"/>
+            </geometry>
+            <material name="white"/>
+        </visual>
+        <visual>
+            <origin xyz="0.144 -0.14515 0.038"/>
+            <geometry>
+                <box size="0.288 0.0025 0.048"/>
+            </geometry>
+            <material name="white"/>
+        </visual>
+        <collision>
+            <origin xyz="0.144 0 0.038"/>
+            <geometry>
+                <box size="0.288 0.2928 0.048"/>
+            </geometry>
+        </collision>
+        <xacro:inertial_box mass="0.5" x="0.288" y="0.2928" z="0.048">
+            <origin xyz="0.144 0 0.038" rpy="0 0 0"/>
         </xacro:inertial_box>
     </link>
@@ -42,9 +98,8 @@
         <material>Gazebo/White</material>
     </gazebo>
-    <!-- FRONT LEFT WHEEL -->
     <joint name="front_left_wheel_joint" type="continuous">
         <parent link="base_link"/>
         <child link="front_left_wheel"/>
-        <origin xyz="0.075 0.175 0" rpy="-${pi/2} 0 0"/>
+        <origin xyz="0.096 0.121 0.038" rpy="-${pi/2} 0 0"/>
         <axis xyz="0 0 1"/>
     </joint>
@@ -52,14 +107,14 @@
         <visual>
             <geometry>
-                <cylinder radius="0.05" length="0.04"/>
-            </geometry>
-            <material name="blue"/>
-        </visual>
-        <collision>
-            <geometry>
-                <cylinder radius="0.05" length="0.04"/>
-            </geometry>
-        </collision>
-        <xacro:inertial_cylinder mass="0.1" length="0.04" radius="0.05">
+                <cylinder radius="0.038" length="0.0408"/>
+            </geometry>
+            <material name="blue"/>
+        </visual>
+        <collision>
+            <geometry>
+                <cylinder radius="0.038" length="0.0408"/>
+            </geometry>
+        </collision>
+        <xacro:inertial_cylinder mass="0.1" length="0.038" radius="0.0408">
             <origin xyz="0 0 0" rpy="0 0 0"/>
         </xacro:inertial_cylinder>
@@ -70,9 +125,8 @@
         <mu2 value="0.0"/>
     </gazebo>
-    <!-- BACK LEFT WHEEL -->
     <joint name="back_left_wheel_joint" type="continuous">
         <parent link="base_link"/>
         <child link="back_left_wheel"/>
-        <origin xyz="-0.075 0.175 0" rpy="-${pi/2} 0 0"/>
+        <origin xyz="-0.096 0.121 0.038" rpy="-${pi/2} 0 0"/>
         <axis xyz="0 0 1"/>
     </joint>
@@ -80,14 +134,14 @@
         <visual>
             <geometry>
-                <cylinder radius="0.05" length="0.04"/>
-            </geometry>
-            <material name="blue"/>
-        </visual>
-        <collision>
-            <geometry>
-                <cylinder radius="0.05" length="0.04"/>
-            </geometry>
-        </collision>
-        <xacro:inertial_cylinder mass="0.1" length="0.04" radius="0.05">
+                <cylinder radius="0.038" length="0.0408"/>
+            </geometry>
+            <material name="blue"/>
+        </visual>
+        <collision>
+            <geometry>
+                <cylinder radius="0.038" length="0.0408"/>
+            </geometry>
+        </collision>
+        <xacro:inertial_cylinder mass="0.1" length="0.038" radius="0.0408">
             <origin xyz="0 0 0" rpy="0 0 0"/>
         </xacro:inertial_cylinder>
@@ -98,9 +152,8 @@
         <mu2 value="0.0"/>
     </gazebo>
-    <!-- FRONT RIGHT WHEEL -->
     <joint name="front_right_wheel_joint" type="continuous">
         <parent link="base_link"/>
         <child link="front_right_wheel"/>
-        <origin xyz="0.075 -0.175 0" rpy="${pi/2} 0 0"/>
+        <origin xyz="0.096 -0.121 0.038" rpy="${pi/2} 0 0"/>
         <axis xyz="0 0 -1"/>
     </joint>
@@ -108,14 +161,14 @@
         <visual>
             <geometry>
-                <cylinder radius="0.05" length="0.04"/>
-            </geometry>
-            <material name="blue"/>
-        </visual>
-        <collision>
-            <geometry>
-                <cylinder radius="0.05" length="0.04"/>
-            </geometry>
-        </collision>
-        <xacro:inertial_cylinder mass="0.1" length="0.04" radius="0.05">
+                <cylinder radius="0.038" length="0.0408"/>
+            </geometry>
+            <material name="blue"/>
+        </visual>
+        <collision>
+            <geometry>
+                <cylinder radius="0.038" length="0.0408"/>
+            </geometry>
+        </collision>
+        <xacro:inertial_cylinder mass="0.1" length="0.038" radius="0.0408">
             <origin xyz="0 0 0" rpy="0 0 0"/>
         </xacro:inertial_cylinder>
@@ -126,9 +179,8 @@
         <mu2 value="0.0"/>
     </gazebo>
-    <!-- BACK RIGHT WHEEL -->
     <joint name="back_right_wheel_joint" type="continuous">
         <parent link="base_link"/>
         <child link="back_right_wheel"/>
-        <origin xyz="-0.075 -0.175 0" rpy="${pi/2} 0 0"/>
+        <origin xyz="-0.096 -0.121 0.038" rpy="${pi/2} 0 0"/>
         <axis xyz="0 0 -1"/>
     </joint>
@@ -136,14 +188,14 @@
         <visual>
             <geometry>
-                <cylinder radius="0.05" length="0.04"/>
-            </geometry>
-            <material name="blue"/>
-        </visual>
-        <collision>
-            <geometry>
-                <cylinder radius="0.05" length="0.04"/>
-            </geometry>
-        </collision>
-        <xacro:inertial_cylinder mass="0.1" length="0.04" radius="0.05">
+                <cylinder radius="0.038" length="0.0408"/>
+            </geometry>
+            <material name="blue"/>
+        </visual>
+        <collision>
+            <geometry>
+                <cylinder radius="0.038" length="0.0408"/>
+            </geometry>
+        </collision>
+        <xacro:inertial_cylinder mass="0.1" length="0.038" radius="0.0408">
             <origin xyz="0 0 0" rpy="0 0 0"/>
         </xacro:inertial_cylinder>

Commit message: camera tuning to better match realsense

File: src/crobot_description/description/depth_camera.xacro (robot description, xacro)
@@ -4,5 +4,5 @@
         <parent link="chassis"/>
         <child link="camera_link"/>
-        <origin xyz="0.305 0 0.038" rpy="0 ${pi/10} 0"/>
+        <origin xyz="0.305 0.12 0.15" rpy="0 ${pi/10} 0"/>
     </joint>
     <link name="camera_link">
@@ -27,5 +27,5 @@
             <update_rate>10</update_rate>
             <camera>
-                <horizontal_fov>1.089</horizontal_fov>
+                <horizontal_fov>1.21126</horizontal_fov>
                 <image>
                     <format>B8G8R8</format>
@@ -34,7 +34,12 @@
                 </image>
                 <clip>
-                    <near>0.05</near>
-                    <far>8.0</far>
+                    <near>0.1</near>
+                    <far>100</far>
                 </clip>
+                <noise>
+                    <type>gaussian</type>
+                    <mean>0</mean>
+                    <stddev>0.007</stddev>
+                </noise>
             </camera>
             <plugin name="camera_controller" filename="libgazebo_ros_camera.so">
