Commit message: got the ros control topics publishing in gazebo

File: src/crobot_description/description/gazebo_control.xacro (robot description, xacro)
@@ -2,5 +2,35 @@
 <robot xmlns:xacro="https://www.ros.org/wiki/xacro">
     <gazebo>
-        <plugin name="gz_ros2_control::GazeboSimROS2ControlPlugin" filename="libgz_ros2_control-system.so">
+        <plugin name="gz::sim::systems::MecanumDrive" filename="libgz-sim8-mecanum-drive-system.so">
+            <!-- ROS 2 integration -->
+            <ros>
+                <namespace>/diff_drive_controller</namespace>
+                <remapping>cmd_vel:=cmd_vel_unstamped</remapping>
+            </ros>
+            <!-- Frames -->
+            <odometry_frame>odom</odometry_frame>
+            <robot_base_frame>base_link</robot_base_frame>
+            <publish_tf>true</publish_tf>
+            <!-- Odometry -->
+            <odometry_rate>50</odometry_rate>
+            <!-- Wheel configuration -->
+            <front_left_wheel>front_left_wheel_joint</front_left_wheel>
+            <front_right_wheel>front_right_wheel_joint</front_right_wheel>
+            <rear_left_wheel>rear_left_wheel_joint</rear_left_wheel>
+            <rear_right_wheel>rear_right_wheel_joint</rear_right_wheel>
+            <!-- Wheel parameters -->
+            <wheel_separation>0.5</wheel_separation> <!-- Distance between left and right wheels -->
+            <wheel_base>0.4</wheel_base> <!-- Distance between front and rear wheels -->
+            <wheel_radius>0.1</wheel_radius> <!-- Radius of the wheels -->
+            <!-- Velocity limits -->
+            <max_linear_velocity>2.0</max_linear_velocity>
+            <max_angular_velocity>1.0</max_angular_velocity>
+        </plugin>
+    </gazebo>
+</robot>
+<!-- <?xml version="1.0"?>
+<robot xmlns:xacro="https://www.ros.org/wiki/xacro">
+    <gazebo>
+       <plugin name="gz::sim::systems::MecanumDrive" filename="libgz_mecanum-drive-system.so" >
             <ros>
                 <namespace>/diff_drive_controller</namespace>
@@ -13,3 +43,3 @@
         </plugin>
     </gazebo>
-</robot>
+</robot> -->

File: src/crobot_description/description/robot_core.xacro (robot description, xacro)
@@ -96,5 +96,9 @@
     </link>
     <gazebo reference="chassis">
-        <material>Gazebo/White</material>
+        <material>
+            <ambient>0.0 0.0 0.0 0.0</ambient> <!--White ? color -->
+            <diffuse>1.0 0.0 0.0 1.0</diffuse>
+            <specular>0.5 0.5 0.5 1.0</specular>
+        </material>
     </gazebo>
     <joint name="front_left_wheel_joint" type="continuous">
@@ -121,5 +125,9 @@
     </link>
     <gazebo reference="front_left_wheel">
-        <material>Gazebo/Blue</material>
+        <material>
+            <ambient>0.0 0.0 0.75 1.0</ambient> <!-- Blue color -->
+            <diffuse>1.0 0.0 0.0 1.0</diffuse>
+            <specular>0.5 0.5 0.5 1.0</specular>
+        </material>
         <mu1 value="0.0"/>
         <mu2 value="0.0"/>
@@ -148,5 +156,9 @@
     </link>
     <gazebo reference="back_left_wheel">
-        <material>Gazebo/Blue</material>
+        <material>
+            <ambient>0.0 0.0 0.75 1.0</ambient> <!-- Blue color -->
+            <diffuse>1.0 0.0 0.0 1.0</diffuse>
+            <specular>0.5 0.5 0.5 1.0</specular>
+        </material>
         <mu1 value="0.0"/>
         <mu2 value="0.0"/>
@@ -175,5 +187,9 @@
     </link>
     <gazebo reference="front_right_wheel">
-        <material>Gazebo/Blue</material>
+        <material>
+             <ambient>0.0 0.0 0.75 1.0</ambient> <!-- Blue color -->
+            <diffuse>1.0 0.0 0.0 1.0</diffuse>
+            <specular>0.5 0.5 0.5 1.0</specular>
+        </material>
         <mu1 value="0.0"/>
         <mu2 value="0.0"/>
@@ -202,5 +218,9 @@
     </link>
     <gazebo reference="back_right_wheel">
-        <material>Gazebo/Blue</material>
+        <material>
+            <ambient>0.0 0.0 0.75 1.0</ambient> <!-- Blue color -->
+            <diffuse>1.0 0.0 0.0 1.0</diffuse>
+            <specular>0.5 0.5 0.5 1.0</specular>
+        </material>
         <mu1 value="0.0"/>
         <mu2 value="0.0"/>

Commit message: mecanum simulated

File: src/crobot_description/description/gazebo_control.xacro (robot description, xacro)
@@ -2,44 +2,28 @@
 <robot xmlns:xacro="https://www.ros.org/wiki/xacro">
     <gazebo>
-        <plugin name="gz::sim::systems::MecanumDrive" filename="libgz-sim8-mecanum-drive-system.so">
+        <!-- <plugin name="gz::sim::systems::MecanumDrive" filename="libgz-sim8-mecanum-drive-system.so"> -->
+        <plugin filename="gz-sim-mecanum-drive-system" name="gz::sim::systems::MecanumDrive">
             <!-- ROS 2 integration -->
-            <ros>
-                <namespace>/diff_drive_controller</namespace>
-                <remapping>cmd_vel:=cmd_vel_unstamped</remapping>
-            </ros>
             <!-- Frames -->
-            <odometry_frame>odom</odometry_frame>
-            <robot_base_frame>base_link</robot_base_frame>
-            <publish_tf>true</publish_tf>
+            <frame_id>odom</frame_id>
+            <child_frame_id>base_link</child_frame_id>
+            <tf_topic>tf</tf_topic>
+            <odom_topic>odom</odom_topic>
+            <topic>cmd_vel</topic>
             <!-- Odometry -->
-            <odometry_rate>50</odometry_rate>
+            <odometry_publish_frequency>50</odometry_publish_frequency>
             <!-- Wheel configuration -->
-            <front_left_wheel>front_left_wheel_joint</front_left_wheel>
-            <front_right_wheel>front_right_wheel_joint</front_right_wheel>
-            <rear_left_wheel>rear_left_wheel_joint</rear_left_wheel>
-            <rear_right_wheel>rear_right_wheel_joint</rear_right_wheel>
+            <front_left_joint>front_left_wheel_joint</front_left_joint>
+            <front_right_joint>front_right_wheel_joint</front_right_joint>
+            <back_left_joint>back_left_wheel_joint</back_left_joint>
+            <back_right_joint>back_right_wheel_joint</back_right_joint>
             <!-- Wheel parameters -->
             <wheel_separation>0.5</wheel_separation> <!-- Distance between left and right wheels -->
-            <wheel_base>0.4</wheel_base> <!-- Distance between front and rear wheels -->
+            <wheelbase>0.4</wheelbase> <!-- Distance between front and rear wheels -->
             <wheel_radius>0.1</wheel_radius> <!-- Radius of the wheels -->
             <!-- Velocity limits -->
-            <max_linear_velocity>2.0</max_linear_velocity>
-            <max_angular_velocity>1.0</max_angular_velocity>
+            <!-- <max_linear_velocity>2.0</max_linear_velocity>
+            <max_angular_velocity>1.0</max_angular_velocity> -->
         </plugin>
     </gazebo>
 </robot>
-<!-- <?xml version="1.0"?>
-<robot xmlns:xacro="https://www.ros.org/wiki/xacro">
-    <gazebo>
-       <plugin name="gz::sim::systems::MecanumDrive" filename="libgz_mecanum-drive-system.so" >
-            <ros>
-                <namespace>/diff_drive_controller</namespace>
-                <remapping>cmd_vel:=cmd_vel_unstamped</remapping>
-            </ros>
-            <odometry_frame>odom</odometry_frame>
-            <odometry_rate>100</odometry_rate>
-            <robot_base_frame>base_link</robot_base_frame>
-            <publish_tf>true</publish_tf>
-        </plugin>
-    </gazebo>
-</robot> -->

File: src/crobot_description/description/robot_core.xacro (robot description, xacro)
@@ -1,4 +1,4 @@
 <?xml version="1.0"?>
-<robot xmlns:xacro="https://www.ros.org/wiki/xacro">
+<robot xmlns:xacro="https://www.ros.org/wiki/xacro" xmlns:gz="http://gazebosim.org/schema">
     <xacro:include filename="inertial_macros.xacro"/>
     <material name="white">
@@ -130,6 +130,15 @@
             <specular>0.5 0.5 0.5 1.0</specular>
         </material>
-        <mu1 value="0.0"/>
-        <mu2 value="0.0"/>
+        <collision>
+            <surface>
+            <friction>
+                <ode>
+                    <mu>1.5</mu>
+                    <mu2>0.0</mu2>
+                    <fdir1 gz:expressed_in="base_link">1 -1 0</fdir1>
+                </ode>
+            </friction>
+            </surface>
+        </collision>
     </gazebo>
     <joint name="back_left_wheel_joint" type="continuous">
@@ -161,6 +170,15 @@
             <specular>0.5 0.5 0.5 1.0</specular>
         </material>
-        <mu1 value="0.0"/>
-        <mu2 value="0.0"/>
+        <collision>
+            <surface>
+            <friction>
+                <ode>
+                <mu>1.5</mu>
+                <mu2>0.0</mu2>
+                <fdir1 gz:expressed_in="base_link">1 1 0</fdir1>
+                </ode>
+            </friction>
+            </surface>
+        </collision>
     </gazebo>
     <joint name="front_right_wheel_joint" type="continuous">
@@ -192,6 +210,15 @@
             <specular>0.5 0.5 0.5 1.0</specular>
         </material>
-        <mu1 value="0.0"/>
-        <mu2 value="0.0"/>
+        <collision>
+            <surface>
+            <friction>
+                <ode>
+                <mu>1.5</mu>
+                <mu2>0.0</mu2>
+                <fdir1 gz:expressed_in="base_link">1 1 0</fdir1>
+                </ode>
+            </friction>
+            </surface>
+        </collision>
     </gazebo>
     <joint name="back_right_wheel_joint" type="continuous">
@@ -223,6 +250,15 @@
             <specular>0.5 0.5 0.5 1.0</specular>
         </material>
-        <mu1 value="0.0"/>
-        <mu2 value="0.0"/>
+        <collision>
+            <surface>
+            <friction>
+                <ode>
+                <mu>1.5</mu>
+                <mu2>0.0</mu2>
+                <fdir1 gz:expressed_in="base_link">1 -1 0</fdir1>
+                </ode>
+            </friction>
+            </surface>
+        </collision>
     </gazebo>
 </robot>
