Commit message: Jayson and domenic are the best, they helped me

File: src/crobot_description/description/camera.xacro (robot description, xacro)
@@ -4,5 +4,5 @@
         <parent link="chassis"/>
         <child link="camera_link"/>
-        <origin xyz="0.305 0 0.08" rpy="0 0 0"/>
+        <origin xyz="0.305 0 0.08" rpy="0 0.1 0"/>
     </joint>
     <link name="camera_link">

Commit message: fixed a few bugs. Ros2 Control and Crobot Navigation are still crashing

File: src/crobot_description/description/camera.xacro (robot description, xacro)
@@ -21,5 +21,9 @@
     <link name="camera_link_optical"/>
     <gazebo reference="camera_link">
-        <material>Gazebo/Red</material>
+        <material>
+            <ambient>1.0 0.0 0.0 1.0</ambient> <!-- Red color -->
+            <diffuse>1.0 0.0 0.0 1.0</diffuse>
+            <specular>0.5 0.5 0.5 1.0</specular>
+        </material>
         <sensor name="camera" type="camera">
             <pose> 0 0 0 0 0 0 </pose>
@@ -27,5 +31,5 @@
             <update_rate>10</update_rate>
             <topic> camera/image_raw</topic>
-            <gz_frame_id>camera_link_optical</gz_frame_id>
+            <gz_frame_id>camera_rgb_frame</gz_frame_id>
             <camera>
                 <camera_info_topic>camera/camera_info</camera_info_topic>

File: src/crobot_description/description/depth_camera.xacro (robot description, xacro)
@@ -21,5 +21,9 @@
     <link name="camera_link_optical"/>
     <gazebo reference="camera_link">
-        <material>Gazebo/Red</material>
+        <material>
+            <ambient>1.0 0.0 0.0 1.0</ambient> <!-- Red color -->
+            <diffuse>1.0 0.0 0.0 1.0</diffuse>
+            <specular>0.5 0.5 0.5 1.0</specular>
+        </material>
         <sensor name="camera" type="depth">
             <pose> 0 0 0 0 0 0 </pose>
@@ -44,5 +48,5 @@
                 </noise>
             </camera>
-            <gz_frame_id>camera_link_optical</gz_frame_id>
+            <frame>camera_link_optical</frame>
             <topic> camera/image_raw_depth</topic>
             <!-- <plugin name="camera_controller" filename="libgazebo_ros_camera.so">

Commit message: reworking some stuff

File: src/crobot_description/description/camera.xacro (robot description, xacro)
@@ -13,4 +13,13 @@
             <material name="orange"/>
         </visual>
+        <collision>
+            <geometry>
+                <box size="0.01 0.03 0.03"/>
+            </geometry>
+        </collision>
+        <inertial>
+            <mass value="0.001"/>
+            <inertia ixx="0.000001" ixy="0" ixz="0" iyy="0.000001" iyz="0" izz="0.000001"/>
+        </inertial>
     </link>
     <joint name="camera_optical" type="fixed">
@@ -20,23 +29,14 @@
     </joint>
     <link name="camera_link_optical"/>
+    <!-- Replace gz:add_camera_sensor with gazebo tag that will convert properly to SDF -->
     <gazebo reference="camera_link">
-        <material>
-            <ambient>1.0 0.0 0.0 1.0</ambient> <!-- Red color -->
-            <diffuse>1.0 0.0 0.0 1.0</diffuse>
-            <specular>0.5 0.5 0.5 1.0</specular>
-        </material>
         <sensor name="camera" type="camera">
-            <pose> 0 0 0 0 0 0 </pose>
-            <visualize>true</visualize>
-            <update_rate>10</update_rate>
-            <topic> camera/image_raw</topic>
-            <gz_frame_id>camera_rgb_frame</gz_frame_id>
+            <pose>0 0 0 0 0 0</pose>
             <camera>
-                <camera_info_topic>camera/camera_info</camera_info_topic>
                 <horizontal_fov>1.089</horizontal_fov>
                 <image>
-                    <format>R8G8B8</format>
                     <width>640</width>
                     <height>480</height>
+                    <format>R8G8B8</format>
                 </image>
                 <clip>
@@ -45,4 +45,8 @@
                 </clip>
             </camera>
+            <always_on>1</always_on>
+            <update_rate>10</update_rate>
+            <visualize>true</visualize>
+            <topic>/camera/image_raw</topic>
         </sensor>
     </gazebo>

File: src/crobot_description/description/depth_camera.xacro (robot description, xacro)
@@ -48,5 +48,5 @@
                 </noise>
             </camera>
-            <frame>camera_link_optical</frame>
+            <gz_frame_id>camera_link_optical</gz_frame_id>
             <topic> camera/image_raw_depth</topic>
             <!-- <plugin name="camera_controller" filename="libgazebo_ros_camera.so">

File: src/crobot_description/description/robot.urdf.xacro (robot description, xacro)
@@ -1,8 +1,9 @@
 <?xml version="1.0"?>
-<robot xmlns:xacro="https://www.ros.org/wiki/xacro" name="robot">
+<!-- <robot xmlns:xacro="https://www.ros.org/wiki/xacro" name="robot"> -->
+<robot name="crobot" xmlns:xacro="http://www.ros.org/wiki/xacro" xmlns:gz="https://github.com/gazebosim/gz_xacro_plugins">
     <xacro:arg name="use_ros2_control" default="true"/>
     <xacro:arg name="sim_mode" default="false"/>
     <xacro:include filename="robot_core.xacro"/>
-    <xacro:include filename="depth_camera.xacro"/>
+    <xacro:include filename="camera.xacro"/>
     <xacro:if value="$(arg use_ros2_control)">
         <xacro:include filename="ros2_control.xacro"/>

File: src/crobot_description/description/robot_core.xacro (robot description, xacro)
@@ -1,4 +1,4 @@
 <?xml version="1.0"?>
-<robot xmlns:xacro="https://www.ros.org/wiki/xacro" xmlns:gz="http://gazebosim.org/schema">
+<robot xmlns:xacro="https://www.ros.org/wiki/xacro" xmlns:gz="https://github.com/gazebosim/gz_xacro_plugins">
     <xacro:include filename="inertial_macros.xacro"/>
     <material name="white">
