Commit message: Ros2 control and gazebo integration for wheels and ankles

File: src/crobot_description/description/robot.urdf.xacro (robot description, xacro)
@@ -2,3 +2,5 @@
 <robot xmlns:xacro="http://www.ros.org/wiki/xacro" name="robot">
   <xacro:include filename="robot_core.xacro"/>
+  <xacro:include filename="ros2_control.xacro"/>
+  <xacro:include filename="gazebo.xacro"/>
 </robot>

File: src/crobot_description/description/robot_core.xacro (robot description, xacro)
@@ -1,4 +1,4 @@
 <?xml version="1.0"?>
-<robot xmlns:xacro="https://www.ros.org/wiki/xacro" name="mars_rover_core">
+<robot xmlns:xacro="https://www.ros.org/wiki/xacro">
   <xacro:include filename="inertial_macros.xacro"/>
   <xacro:include filename="materials.xacro"/>
@@ -199,53 +199,3 @@
   <xacro:ankle_and_wheel name="rear_left"  xpos="${x_rear}" ypos="${y_left}"  is_omni="false"/>
   <xacro:ankle_and_wheel name="rear_right" xpos="${x_rear}" ypos="${y_right}" is_omni="false"/>
-  <ros2_control name="GazeboSystem" type="system">
-    <hardware>
-      <plugin>gz_ros2_control/GazeboSystem</plugin>
-    </hardware>
-    <joint name="front_left_ankle_joint">
-      <command_interface name="position"/>
-      <state_interface   name="position"/>
-    </joint>
-    <joint name="front_left_wheel_joint">
-      <command_interface name="velocity"/>
-      <state_interface   name="velocity"/>
-    </joint>
-    <joint name="front_right_ankle_joint">
-      <command_interface name="position"/>
-      <state_interface   name="position"/>
-    </joint>
-    <joint name="front_right_wheel_joint">
-      <command_interface name="velocity"/>
-      <state_interface   name="velocity"/>
-    </joint>
-    <joint name="mid_left_wheel_joint">
-      <command_interface name="velocity"/>
-      <state_interface   name="velocity"/>
-    </joint>
-    <joint name="mid_right_wheel_joint">
-      <command_interface name="velocity"/>
-      <state_interface   name="velocity"/>
-    </joint>
-    <joint name="rear_left_ankle_joint">
-      <command_interface name="position"/>
-      <state_interface   name="position"/>
-    </joint>
-    <joint name="rear_left_wheel_joint">
-      <command_interface name="velocity"/>
-      <state_interface   name="velocity"/>
-    </joint>
-    <joint name="rear_right_ankle_joint">
-      <command_interface name="position"/>
-      <state_interface   name="position"/>
-    </joint>
-    <joint name="rear_right_wheel_joint">
-      <command_interface name="velocity"/>
-      <state_interface   name="velocity"/>
-    </joint>
-  </ros2_control>
-  <gazebo>
-    <plugin filename="gz-sim-ros2-control-system" name="gz_ros2_control">
-      <parameters>$(find gazebo_launch)/config/minimal.yaml</parameters>
-    </plugin>
-  </gazebo>
 </robot>
