Commit message: A semi working simulation with a semi ok map

File: src/crobot_description/description/lidar.xacro (robot description, xacro)
@@ -4,5 +4,5 @@
         <parent link="base_link"/>
         <child link="laser_frame"/>
-        <origin xyz="0.122 0 0.212" rpy="0 0 0"/>
+        <origin xyz="0.122 0 0.100" rpy="0 0 0"/>
     </joint>
     <link name="laser_frame">

File: src/crobot_description/description/ros2_control.xacro (robot description, xacro)
@@ -3,6 +3,9 @@
   <ros2_control name="Crobot" type="system">
     <hardware>
+      <!-- <xacro:if value="$(arg sim_mode)">
+        <plugin>gz_ros2_control/GazeboSimSystem</plugin>
+      </xacro:if> -->
       <xacro:if value="$(arg sim_mode)">
-        <plugin>gz_ros2_control/GazeboSimSystem</plugin>
+        <plugin>ign_ros2_control/IgnitionSystem</plugin>
       </xacro:if>
       <xacro:unless value="$(arg sim_mode)">
@@ -72,7 +75,17 @@
   <xacro:if value="$(arg sim_mode)">
     <gazebo>
-      <plugin filename="gz_ros2_control-system" name="gz_ros2_control::GazeboSimROS2ControlPlugin">
+      <!-- <plugin filename="gz_ros2_control-system" name="gz_ros2_control::GazeboSimROS2ControlPlugin">
         <parameters>$(find crobot_controller)/config/gazebo_ros2_control_use_sim.yaml</parameters>
+      </plugin> -->
+      <plugin filename="ign_ros2_control-system"
+            name="ign_ros2_control::IgnitionROS2ControlPlugin">
+      <parameters>$(find crobot_controller)/config/gazebo_ros2_control_use_sim.yaml</parameters>
       </plugin>
+      <plugin filename="ignition-gazebo-odometry-publisher-system"
+            name="ignition::gazebo::systems::OdometryPublisher">
+      <odom_frame>odom</odom_frame>
+      <robot_base_frame>base_link</robot_base_frame>
+      <odom_publish_frequency>50</odom_publish_frequency>
+    </plugin>
     </gazebo>
   </xacro:if>
