Commit message: gazebo world files

File: src/crobot_description/description/robot_core.xacro (robot description, xacro)
@@ -23,5 +23,5 @@
     <link name="chassis">
         <visual>
-            <origin xyz="0.144 0 0.038"/>
+            <origin xyz="-0.456 -0.9 0.038"/>
             <geometry>
                 <box size="0.096 0.168 0.048"/>
@@ -30,5 +30,5 @@
         </visual>
         <visual>
-            <origin xyz="0.144 0.09 0.038"/>
+            <origin xyz="-0.456 -0.81 0.038"/>
             <geometry>
                 <box size="0.288 0.012 0.048"/>
@@ -37,5 +37,5 @@
         </visual>
         <visual>
-            <origin xyz="0.144 -0.09 0.038"/>
+            <origin xyz="-0.456 -0.99 0.038"/>
             <geometry>
                 <box size="0.288 0.012 0.048"/>
@@ -44,33 +44,33 @@
         </visual>
         <visual>
-            <origin xyz="0.00125 0.11995 0.038"/>
-            <geometry>
-                <box size="0.0025 0.0479 0.048"/>
-            </geometry>
-            <material name="white"/>
-        </visual>
-        <visual>
-            <origin xyz="0.00125 -0.11995 0.038"/>
-            <geometry>
-                <box size="0.0025 0.0479 0.048"/>
-            </geometry>
-            <material name="white"/>
-        </visual>
-        <visual>
-            <origin xyz="0.28675 0.11995 0.038"/>
-            <geometry>
-                <box size="0.0025 0.0479 0.048"/>
-            </geometry>
-            <material name="white"/>
-        </visual>
-        <visual>
-            <origin xyz="0.28675 -0.11995 0.038"/>
-            <geometry>
-                <box size="0.0025 0.0479 0.048"/>
-            </geometry>
-            <material name="white"/>
-        </visual>
-        <visual>
-            <origin xyz="0.144 0.14515 0.038"/>
+            <origin xyz="-0.59875 -0.78005 0.038"/>
+            <geometry>
+                <box size="0.0025 0.0479 0.048"/>
+            </geometry>
+            <material name="white"/>
+        </visual>
+        <visual>
+            <origin xyz="-0.59875 -1.01995 0.038"/>
+            <geometry>
+                <box size="0.0025 0.0479 0.048"/>
+            </geometry>
+            <material name="white"/>
+        </visual>
+        <visual>
+            <origin xyz="-0.31325 -0.78005 0.038"/>
+            <geometry>
+                <box size="0.0025 0.0479 0.048"/>
+            </geometry>
+            <material name="white"/>
+        </visual>
+        <visual>
+            <origin xyz="-0.31325 -1.01995 0.038"/>
+            <geometry>
+                <box size="0.0025 0.0479 0.048"/>
+            </geometry>
+            <material name="white"/>
+        </visual>
+        <visual>
+            <origin xyz="-0.456 -0.75485 0.038"/>
             <geometry>
                 <box size="0.288 0.0025 0.048"/>
@@ -79,5 +79,5 @@
         </visual>
         <visual>
-            <origin xyz="0.144 -0.14515 0.038"/>
+            <origin xyz="-0.456 -1.05485 0.038"/>
             <geometry>
                 <box size="0.288 0.0025 0.048"/>

Commit message: robot spawns in new gazebo

File: src/crobot_description/description/robot_core.xacro (robot description, xacro)
@@ -199,11 +199,53 @@
   <xacro:ankle_and_wheel name="rear_left"  xpos="${x_rear}" ypos="${y_left}"  is_omni="false"/>
   <xacro:ankle_and_wheel name="rear_right" xpos="${x_rear}" ypos="${y_right}" is_omni="false"/>
-  <!-- Gazebo visual hint (optional) -->
-  <gazebo reference="chassis">
-    <material>
-      <ambient>0 0 0 0</ambient>
-      <diffuse>1 1 1 1</diffuse>
-      <specular>0.5 0.5 0.5 1</specular>
-    </material>
+  <ros2_control name="GazeboSystem" type="system">
+    <hardware>
+      <plugin>gz_ros2_control/GazeboSystem</plugin>
+    </hardware>
+    <joint name="front_left_ankle_joint">
+      <command_interface name="position"/>
+      <state_interface   name="position"/>
+    </joint>
+    <joint name="front_left_wheel_joint">
+      <command_interface name="velocity"/>
+      <state_interface   name="velocity"/>
+    </joint>
+    <joint name="front_right_ankle_joint">
+      <command_interface name="position"/>
+      <state_interface   name="position"/>
+    </joint>
+    <joint name="front_right_wheel_joint">
+      <command_interface name="velocity"/>
+      <state_interface   name="velocity"/>
+    </joint>
+    <joint name="mid_left_wheel_joint">
+      <command_interface name="velocity"/>
+      <state_interface   name="velocity"/>
+    </joint>
+    <joint name="mid_right_wheel_joint">
+      <command_interface name="velocity"/>
+      <state_interface   name="velocity"/>
+    </joint>
+    <joint name="rear_left_ankle_joint">
+      <command_interface name="position"/>
+      <state_interface   name="position"/>
+    </joint>
+    <joint name="rear_left_wheel_joint">
+      <command_interface name="velocity"/>
+      <state_interface   name="velocity"/>
+    </joint>
+    <joint name="rear_right_ankle_joint">
+      <command_interface name="position"/>
+      <state_interface   name="position"/>
+    </joint>
+    <joint name="rear_right_wheel_joint">
+      <command_interface name="velocity"/>
+      <state_interface   name="velocity"/>
+    </joint>
+  </ros2_control>
+  <gazebo>
+    <plugin filename="gz-sim-ros2-control-system" name="gz_ros2_control">
+      <parameters>$(find gazebo_launch)/config/minimal.yaml</parameters>
+    </plugin>
   </gazebo>
 </robot>

Commit message: More hardwareinterface plugin - NEED READ WRITE

File: src/crobot_description/description/robot_core.xacro (robot description, xacro)
@@ -16,5 +16,5 @@
   <xacro:property name="x_front" value="${body_length/2.0 - 0.018}"/>
   <xacro:property name="x_mid"   value="0.0"/>
-  <xacro:property name="x_rear"  value="${-body_length/2.0 + 0.018}"/>
+  <xacro:property name="x_back"  value="${-body_length/2.0 + 0.018}"/>
   <xacro:property name="y_left"  value="${body_width/2.0 - 0.01}"/>
   <xacro:property name="y_right" value="${-body_width/2.0 + 0.01}"/>
@@ -196,6 +196,6 @@
     <axis xyz="0 1 0"/>
   </joint>
-  <!-- REAR LEFT / RIGHT -->
-  <xacro:ankle_and_wheel name="rear_left"  xpos="${x_rear}" ypos="${y_left}"  is_omni="false"/>
-  <xacro:ankle_and_wheel name="rear_right" xpos="${x_rear}" ypos="${y_right}" is_omni="false"/>
+  <!-- BACK LEFT / RIGHT -->
+  <xacro:ankle_and_wheel name="back_left"  xpos="${x_back}" ypos="${y_left}"  is_omni="false"/>
+  <xacro:ankle_and_wheel name="back_right" xpos="${x_back}" ypos="${y_right}" is_omni="false"/>
 </robot>

File: src/crobot_description/description/ros2_control.xacro (robot description, xacro)
@@ -4,9 +4,21 @@
     <hardware>
       <xacro:if value="$(arg sim_mode)">
-        <!-- TODO: Determine if this gazebo plugin is right -->
         <plugin>gz_ros2_control/GazeboSimSystem</plugin>
       </xacro:if>
       <xacro:unless value="$(arg sim_mode)">
         <plugin>crobot_hardware/CrobotHardware</plugin>
+        <param name="front_left_wheel_name">front_left_wheel_joint</param>
+        <param name="front_right_wheel_name">front_right_wheel_joint</param>
+        <param name="back_left_wheel_name">back_left_wheel_joint</param>
+        <param name="back_right_wheel_name">back_right_wheel_joint</param>
+        <param name="front_left_ankle_name">front_left_ankle_joint</param>
+        <param name="front_right_ankle_name">front_right_ankle_joint</param>
+        <param name="back_left_ankle_name">back_left_ankle_joint</param>
+        <param name="back_right_ankle_name">back_right_ankle_joint</param>
+        <!-- TODO: Confirm parameters -->
+        <param name="loop_rate">30.0</param>
+        <param name="dev">/dev/ttyTHS1</param>
+        <param name="baud_rate">115200</param>
+        <param name="timeout_ms">1000</param>
       </xacro:unless>
     </hardware>
@@ -15,38 +27,42 @@
       <state_interface   name="position"/>
     </joint>
-    <joint name="front_left_wheel_joint">
-      <command_interface name="velocity"/>
-      <state_interface   name="velocity"/>
-    </joint>
     <joint name="front_right_ankle_joint">
       <command_interface name="position"/>
       <state_interface   name="position"/>
     </joint>
-    <joint name="front_right_wheel_joint">
-      <command_interface name="velocity"/>
-      <state_interface   name="velocity"/>
-    </joint>
-    <joint name="mid_left_wheel_joint">
-      <command_interface name="velocity"/>
-      <state_interface   name="velocity"/>
-    </joint>
-    <joint name="mid_right_wheel_joint">
-      <command_interface name="velocity"/>
-      <state_interface   name="velocity"/>
-    </joint>
-    <joint name="rear_left_ankle_joint">
+    <joint name="back_left_ankle_joint">
       <command_interface name="position"/>
       <state_interface   name="position"/>
     </joint>
-    <joint name="rear_left_wheel_joint">
-      <command_interface name="velocity"/>
-      <state_interface   name="velocity"/>
-    </joint>
-    <joint name="rear_right_ankle_joint">
+    <joint name="back_right_ankle_joint">
       <command_interface name="position"/>
       <state_interface   name="position"/>
     </joint>
-    <joint name="rear_right_wheel_joint">
-      <command_interface name="velocity"/>
+    <joint name="front_left_wheel_joint">
+      <command_interface name="velocity">
+        <param name="min">-10.0</param>
+        <param name="max">10.0</param>
+      </command_interface>
+      <state_interface   name="velocity"/>
+    </joint>
+    <joint name="front_right_wheel_joint">
+      <command_interface name="velocity">
+        <param name="min">-10.0</param>
+        <param name="max">10.0</param>
+      </command_interface>
+      <state_interface   name="velocity"/>
+    </joint>
+    <joint name="back_left_wheel_joint">
+      <command_interface name="velocity">
+        <param name="min">-10.0</param>
+        <param name="max">10.0</param>
+      </command_interface>
+      <state_interface   name="velocity"/>
+    </joint>
+    <joint name="back_right_wheel_joint">
+      <command_interface name="velocity">
+        <param name="min">-10.0</param>
+        <param name="max">10.0</param>
+      </command_interface>
       <state_interface   name="velocity"/>
     </joint>

Commit message: more accurate sim variables

File: src/crobot_description/description/robot_core.xacro (robot description, xacro)
@@ -4,9 +4,9 @@
   <xacro:include filename="materials.xacro"/>
   <!-- Parameters -->
-  <xacro:property name="body_length"  value="0.28"/>
-  <xacro:property name="body_width"   value="0.24"/>
+  <xacro:property name="body_length"  value="0.3048"/>
+  <xacro:property name="body_width"   value="0.25"/>
   <xacro:property name="body_height"  value="0.10"/>
   <xacro:property name="drivetrain_height" value="0.02"/>
-  <xacro:property name="wheel_radius" value="0.038"/>
+  <xacro:property name="wheel_radius" value="0.035"/>
   <xacro:property name="wheel_width"  value="0.0408"/>
   <xacro:property name="wheel_mass"   value="0.15"/>
@@ -14,9 +14,9 @@
   <xacro:property name="chassis_mass" value="2.0"/>
   <xacro:property name="ankle_mass"   value="0.05"/>
-  <xacro:property name="x_front" value="${body_length/2.0 - 0.018}"/>
+  <xacro:property name="x_front" value="0.115"/>
   <xacro:property name="x_mid"   value="0.0"/>
-  <xacro:property name="x_back"  value="${-body_length/2.0 + 0.018}"/>
-  <xacro:property name="y_left"  value="${body_width/2.0 - 0.01}"/>
-  <xacro:property name="y_right" value="${-body_width/2.0 + 0.01}"/>
+  <xacro:property name="x_back"  value="-0.115"/>
+  <xacro:property name="y_left"  value="0.075"/>
+  <xacro:property name="y_right" value="-0.075"/>
   <!-- base_link is the robot origin (center of chassis) -->
   <link name="base_link"/>
@@ -196,4 +196,12 @@
     <axis xyz="0 1 0"/>
   </joint>
+  <gazebo reference="mid_left_wheel">
+    <mu1>1.0</mu1>
+    <mu2>0.0</mu2>
+  </gazebo>
+  <gazebo reference="mid_right_wheel">
+    <mu1>1.0</mu1>
+    <mu2>0.0</mu2>
+  </gazebo>
   <!-- BACK LEFT / RIGHT -->
   <xacro:ankle_and_wheel name="back_left"  xpos="${x_back}" ypos="${y_left}"  is_omni="false"/>

File: src/crobot_description/description/ros2_control.xacro (robot description, xacro)
@@ -42,29 +42,17 @@
     </joint>
     <joint name="front_left_wheel_joint">
-      <command_interface name="velocity">
-        <param name="min">-10.0</param>
-        <param name="max">10.0</param>
-      </command_interface>
+      <command_interface name="velocity"/>
       <state_interface   name="velocity"/>
     </joint>
     <joint name="front_right_wheel_joint">
-      <command_interface name="velocity">
-        <param name="min">-10.0</param>
-        <param name="max">10.0</param>
-      </command_interface>
+      <command_interface name="velocity"/>
       <state_interface   name="velocity"/>
     </joint>
     <joint name="back_left_wheel_joint">
-      <command_interface name="velocity">
-        <param name="min">-10.0</param>
-        <param name="max">10.0</param>
-      </command_interface>
+      <command_interface name="velocity"/>
       <state_interface   name="velocity"/>
     </joint>
     <joint name="back_right_wheel_joint">
-      <command_interface name="velocity">
-        <param name="min">-10.0</param>
-        <param name="max">10.0</param>
-      </command_interface>
+      <command_interface name="velocity"/>
       <state_interface   name="velocity"/>
     </joint>

Commit message: wheel positions and camera joint

File: src/crobot_description/description/robot_core.xacro (robot description, xacro)
@@ -21,4 +21,5 @@
   <!-- base_link is the robot origin (center of chassis) -->
   <link name="base_link"/>
+  <link name="camera_link"/>
   <!-- CHASSIS (link frame at its center) -->
   <link name="chassis">
@@ -47,4 +48,11 @@
     <child  link="chassis"/>
     <origin xyz="0 0 0" rpy="0 0 0"/>
+  </joint>
+  <joint name="camera_joint" type="fixed">
+    <parent link="base_link"/>
+    <child link="camera_link"/>
+    <!-- TODO: CHANGE THIS!!!!!!!!!!!!!!!!!!!-->
+    <origin xyz="0 0 0.5" rpy="0 0 0"/>
+    <!-- !!!!!!!!!!!!!!!!!!!!!!!!!!!!!!!!!!!!!!!!-->
   </joint>
   <!-- MACRO: ankle mount and wheel.

File: src/crobot_description/description/ros2_control.xacro (robot description, xacro)
@@ -44,16 +44,20 @@
       <command_interface name="velocity"/>
       <state_interface   name="velocity"/>
+      <state_interface   name="position"/>
     </joint>
     <joint name="front_right_wheel_joint">
       <command_interface name="velocity"/>
       <state_interface   name="velocity"/>
+      <state_interface   name="position"/>
     </joint>
     <joint name="back_left_wheel_joint">
       <command_interface name="velocity"/>
       <state_interface   name="velocity"/>
+      <state_interface   name="position"/>
     </joint>
     <joint name="back_right_wheel_joint">
       <command_interface name="velocity"/>
       <state_interface   name="velocity"/>
+      <state_interface   name="position"/>
     </joint>
     <joint name="sweeper_joint">

Commit message: nvblox running :) cant see it

File: src/crobot_description/description/robot_core.xacro (robot description, xacro)
@@ -21,5 +21,5 @@
   <!-- base_link is the robot origin (center of chassis) -->
   <link name="base_link"/>
-  <link name="camera_link"/>
+  <link name="camera0_link"/>
   <!-- CHASSIS (link frame at its center) -->
   <link name="chassis">
@@ -51,5 +51,5 @@
   <joint name="camera_joint" type="fixed">
     <parent link="base_link"/>
-    <child link="camera_link"/>
+    <child link="camera0_link"/>
     <!-- TODO: CHANGE THIS!!!!!!!!!!!!!!!!!!!-->
     <origin xyz="0 0 0.5" rpy="0 0 0"/>

Commit message: IDK Changes from wtv Olivia did?

File: src/crobot_description/description/robot_core.xacro (robot description, xacro)
@@ -53,5 +53,5 @@
     <child link="camera0_link"/>
     <!-- TODO: CHANGE THIS!!!!!!!!!!!!!!!!!!!-->
-    <origin xyz="0 0 0.5" rpy="0 0 0"/>
+    <origin xyz="0.16 0 0.02" rpy="0 0 0"/>
     <!-- !!!!!!!!!!!!!!!!!!!!!!!!!!!!!!!!!!!!!!!!-->
   </joint>

Commit message: changing nvblox params

File: src/crobot_description/description/robot_core.xacro (robot description, xacro)
@@ -53,5 +53,5 @@
     <child link="camera0_link"/>
     <!-- TODO: CHANGE THIS!!!!!!!!!!!!!!!!!!!-->
-    <origin xyz="0.16 0 0.02" rpy="0 0 0"/>
+    <origin xyz="0.16 0 0.03" rpy="0 0 0"/>
     <!-- !!!!!!!!!!!!!!!!!!!!!!!!!!!!!!!!!!!!!!!!-->
   </joint>

Commit message: removed middle wheel from gazebo
enabled pointcloud scan from realsense for scan data

File: src/crobot_description/description/robot_core.xacro (robot description, xacro)
@@ -121,5 +121,5 @@
        and a wheel joint from that mount to the wheel where origin=0 0 0. -->
   <!-- MID LEFT -->
-  <link name="mid_left_mount">
+  <!-- <link name="mid_left_mount">
     <visual>
       <origin xyz="0 0 ${-drivetrain_height / 2.0}" rpy="0 0 0"/>
@@ -161,7 +161,7 @@
     <origin xyz="0 0 ${-drivetrain_height - wheel_radius}" rpy="0 0 0"/>
     <axis xyz="0 1 0"/>
-  </joint>
+  </joint> -->
   <!-- MID RIGHT -->
-  <link name="mid_right_mount">
+  <!-- <link name="mid_right_mount">
     <visual>
       <origin xyz="0 0 ${-drivetrain_height / 2.0}" rpy="0 0 0"/>
@@ -203,6 +203,6 @@
     <origin xyz="0 0 ${-drivetrain_height - wheel_radius}" rpy="0 0 0"/>
     <axis xyz="0 1 0"/>
-  </joint>
-  <gazebo reference="mid_left_wheel">
+  </joint> -->
+  <!-- <gazebo reference="mid_left_wheel">
     <mu1>0.0</mu1>
     <mu2>0.0</mu2>
@@ -211,5 +211,5 @@
     <mu1>0.0</mu1>
     <mu2>0.0</mu2>
-  </gazebo>
+  </gazebo> -->
   <!-- BACK LEFT / RIGHT -->
   <xacro:ankle_and_wheel name="back_left"  xpos="${x_back}" ypos="${y_left}"  is_omni="false"/>

Commit message: robot is always extended forward with sweeper

File: src/crobot_description/description/robot_core.xacro (robot description, xacro)
@@ -26,14 +26,14 @@
     <visual>
       <!-- visual origin relative to chassis link frame (center) -->
-      <origin xyz="0 0 0" rpy="0 0 0"/>
-      <geometry>
-        <box size="${body_length} ${body_width} ${body_height}"/>
+      <origin xyz="0.04445 0 0" rpy="0 0 0"/>
+      <geometry>
+        <box size="0.4 ${body_width} ${body_height}"/>
       </geometry>
       <material name="white"/>
     </visual>
     <collision>
-      <origin xyz="0 0 0" rpy="0 0 0"/>
-      <geometry>
-        <box size="${body_length} ${body_width} ${body_height}"/>
+      <origin xyz="0.04445 0 0" rpy="0 0 0"/>
+      <geometry>
+        <box size="0.4 ${body_width} ${body_height}"/>
       </geometry>
     </collision>
