Commit message: crobot bringup launch working for custom hardware interface

File: src/crobot_description/description/ros2_control.xacro (robot description, xacro)
@@ -4,16 +4,16 @@
         <ros2_control name="Crobot" type="system">
             <hardware>
-                <plugin>diff_drive_controller/DiffDriveController</plugin>
+                <plugin>crobot_hardware/CrobotHardware</plugin>
                 <param name="front_left_wheel_name">front_left_wheel_joint</param>
                 <param name="back_left_wheel_name">back_left_wheel_joint</param>
                 <param name="front_right_wheel_name">front_right_wheel_joint</param>
                 <param name="back_right_wheel_name">back_right_wheel_joint</param>
-                <param name="loop_rate">30</param>
+                <param name="loop_rate">30.0</param>
                 <param name="dev">/dev/ttyACM0</param>
                 <param name="baud_rate">57600</param>
-                <param name="timeout">1000</param>
+                <param name="timeout_ms">1000</param>
                 <param name="enc_counts_per_rev">3450</param>
             </hardware>
-            <joint name="front_left_wheel_joint">
+            <!-- <joint name="front_left_wheel_joint">
                 <command_interface name="velocity">
                     <param name="min">-10</param>
@@ -46,5 +46,5 @@
                 <state_interface name="velocity"/>
                 <state_interface name="position"/>
-            </joint>
+            </joint> -->
         </ros2_control>
     </xacro:unless>
@@ -87,10 +87,10 @@
             </joint>
         </ros2_control>
+        <gazebo>
+            <plugin name="gazebo_ros2_control" filename="libgazebo_ros2_control.so">
+                <parameters>$(find crobot_controller)/config/ros2_control.yaml</parameters>
+                <parameters>$(find crobot_controller)/config/gazebo_ros2_control_use_sim.yaml</parameters>
+            </plugin>
+        </gazebo>
     </xacro:if>
-    <gazebo>
-        <plugin name="gazebo_ros2_control" filename="libgazebo_ros2_control.so">
-            <parameters>$(find crobot_controller)/config/ros2_control.yaml</parameters>
-            <parameters>$(find crobot_controller)/config/gazebo_ros2_control_use_sim.yaml</parameters>
-        </plugin>
-    </gazebo>
 </robot>

Commit message: hardware bringup setup, need to implement controller and hardware interface

File: src/crobot_description/description/ros2_control.xacro (robot description, xacro)
@@ -15,11 +15,11 @@
                 <param name="enc_counts_per_rev">3450</param>
             </hardware>
-            <!-- <joint name="front_left_wheel_joint">
+            <joint name="front_left_wheel_joint">
                 <command_interface name="velocity">
                     <param name="min">-10</param>
                     <param name="max">10</param>
                 </command_interface>
+                <state_interface name="position"/>
                 <state_interface name="velocity"/>
-                <state_interface name="position"/>
             </joint>
             <joint name="front_right_wheel_joint">
@@ -28,6 +28,6 @@
                     <param name="max">10</param>
                 </command_interface>
+                <state_interface name="position"/>
                 <state_interface name="velocity"/>
-                <state_interface name="position"/>
             </joint>
             <joint name="back_left_wheel_joint">
@@ -36,6 +36,6 @@
                     <param name="max">10</param>
                 </command_interface>
+                <state_interface name="position"/>
                 <state_interface name="velocity"/>
-                <state_interface name="position"/>
             </joint>
             <joint name="back_right_wheel_joint">
@@ -44,7 +44,7 @@
                     <param name="max">10</param>
                 </command_interface>
+                <state_interface name="position"/>
                 <state_interface name="velocity"/>
-                <state_interface name="position"/>
-            </joint> -->
+            </joint>
         </ros2_control>
     </xacro:unless>

Commit message: temp temp crobot_controller (thanks claude)

File: src/crobot_description/description/ros2_control.xacro (robot description, xacro)
@@ -16,4 +16,5 @@
         <param name="back_left_ankle_name">back_left_ankle_joint</param>
         <param name="back_right_ankle_name">back_right_ankle_joint</param>
+        <param name="sweeper_name">sweeper_joint</param>
         <!-- TODO: Confirm parameters -->
         <param name="loop_rate">30.0</param>
@@ -67,4 +68,8 @@
       <state_interface   name="velocity"/>
     </joint>
+    <joint name="sweeper_joint">
+      <command_interface name="position"/>
+      <state_interface   name="position"/>
+    </joint>
   </ros2_control>
   <xacro:if value="$(arg sim_mode)">

Commit message: no sweeper yet

File: src/crobot_description/description/ros2_control.xacro (robot description, xacro)
@@ -16,5 +16,5 @@
         <param name="back_left_ankle_name">back_left_ankle_joint</param>
         <param name="back_right_ankle_name">back_right_ankle_joint</param>
-        <param name="sweeper_name">sweeper_joint</param>
+        <!-- <param name="sweeper_name">sweeper_joint</param> -->
         <!-- TODO: Confirm parameters -->
         <param name="loop_rate">30.0</param>
@@ -68,8 +68,8 @@
       <state_interface   name="velocity"/>
     </joint>
-    <joint name="sweeper_joint">
+    <!-- <joint name="sweeper_joint">
       <command_interface name="position"/>
       <state_interface   name="position"/>
-    </joint>
+    </joint> -->
   </ros2_control>
   <xacro:if value="$(arg sim_mode)">

Commit message: expose winch and sweeper in ros2 control

File: src/crobot_description/description/ros2_control.xacro (robot description, xacro)
@@ -68,8 +68,12 @@
       <state_interface   name="velocity"/>
     </joint>
-    <!-- <joint name="sweeper_joint">
+    <joint name="sweeper_joint">
       <command_interface name="position"/>
       <state_interface   name="position"/>
-    </joint> -->
+    </joint>
+    <joint name="winch_joint">
+      <command_interface name="velocity"/>
+      <state_interface   name="velocity"/>
+    </joint>
   </ros2_control>
   <xacro:if value="$(arg sim_mode)">

Commit message: use imu for ang z

File: src/crobot_description/description/ros2_control.xacro (robot description, xacro)
@@ -19,4 +19,5 @@
         <param name="back_left_ankle_name">back_left_ankle_joint</param>
         <param name="back_right_ankle_name">back_right_ankle_joint</param>
+        <param name="imu_name">base_to_imu_joint</param>
         <param name="sweeper_name">sweeper_joint</param>
         <param name="winch_name">winch_joint</param>
@@ -74,4 +75,7 @@
       <!-- <state_interface   name="velocity"/> -->
     </joint>
+    <joint name="base_to_imu_joint">
+      <state_interface   name="velocity"/>
+    </joint>
   </ros2_control>
   <xacro:if value="$(arg sim_mode)">

Commit message: this should build now?

File: src/crobot_description/description/ros2_control.xacro (robot description, xacro)
@@ -22,4 +22,7 @@
         <param name="sweeper_name">sweeper_joint</param>
         <param name="winch_name">winch_joint</param>
+        <joint name="flagdropper_joint">
+          <command_interface name="velocity"/>
+        </joint>
         <!-- TODO: Confirm parameters -->
         <param name="loop_rate">30.0</param>
